File: freezanz-level-io/freezanz-level-io.kicad_pcb (KiCad board)
At the start: 2 copper layers, 90 x 50 mm, 51 parts, among them J1 IDC 2x4 <- Freezanz J3, J11 S1, J12 S2, J13 S3, J14 S4, J15 S5, J16 S6, J17 S7, J18 S8, J21 I2C EXP1, J22 I2C EXP2, J23 I2C EXP3, J3 MCP LEFT, J4 MCP RIGHT, J6 MCP PORT B, J7 INT / SPARE, J8 GPIO5 OUT, J9 GPIO15 OUT

Commit message: Fixed SVG, production board sent via kicad
Parts:
- moved H1 4.21 mm to (100.5, 60.5)
- moved H2 3.62 mm to (100.5, 108.5)
- moved H3 3.53 mm to (188.5, 60.5)
- moved H4 2.85 mm to (188.5, 108.5)
Other:
- board size 90 x 50 mm -> 93 x 53 mm

Commit message: Pushing v2 version of the breakout board
Parts:
- added D2: LED, LED_THT:LED_D5.0mm, F.Cu at (184.7, 68.2)
- added R6: 470R, Resistor_THT:R_Axial_DIN0207_L6.3mm_D2.5mm_P7.62mm_Horizontal, F.Cu at (164.4, 66.1)
- added R7: 470R, Resistor_THT:R_Axial_DIN0207_L6.3mm_D2.5mm_P7.62mm_Horizontal, F.Cu at (164.4, 69.7)
- added R8: 10k, Resistor_THT:R_Axial_DIN0207_L6.3mm_D2.5mm_P7.62mm_Horizontal, F.Cu at (180.7, 70.4)
- F1: value F 12v - 500mA 5x20 -> F200mA (F=fast) 5x20
- J6: value MCP PORT B -> PORT B
- moved JP2 24.6 mm to (163.7, 60.9)
- moved J21 10.6 mm to (135.4, 62.7)
- moved J22 10.6 mm to (121.4, 62.7)
- moved J23 10.6 mm to (107.4, 62.7)
- moved C3 10.6 mm to (149.8, 67.4)
- moved C4 10.6 mm to (148.0, 61.8)
- moved J11 7.50 mm to (110.5, 71.0), turned to 180 degrees
- moved J12 7.50 mm to (126.5, 75.0), turned to 180 degrees
- moved J13 7.50 mm to (110.5, 79.0), turned to 180 degrees
- moved J14 7.50 mm to (126.5, 83.0), turned to 180 degrees
- moved J15 7.50 mm to (110.5, 87.0), turned to 180 degrees
- moved J16 7.50 mm to (126.5, 91.0), turned to 180 degrees
- moved J17 7.50 mm to (110.5, 95.0), turned to 180 degrees
- moved J18 7.50 mm to (126.5, 99.0), turned to 180 degrees
- moved R2 4.94 mm to (166.0, 97.1)
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Connections:
- net /GPB0 renamed /A0
- net /GPB1 renamed /A1
- net /GPB2 renamed /A2
- net /GPB3 renamed /A3
- net /GPB4 renamed /A4
- net /GPB5 renamed /A5
- net /GPB6 renamed /A6
- net /GPB7 renamed /A7
- net /IO1 renamed /B0
- net /IO2 renamed /B1
- net /IO3 renamed /B2
- net /IO4 renamed /B3
- net /IO5 renamed /B4
- net /IO6 renamed /B5
- net /IO7 renamed /B6
- net /IO8 renamed /B7
- J1 pad 5: /SDA -> /SDA_J1
- J1 pad 7: /SCL -> /SCL_J1
- J11 pad 1: /SENS_M -> /+12V
- J11 pad 2: /GND -> /SIG1
- J11 pad 3: /SIG1 -> /GND
- J11 pad 4: /+12V -> /SENS_M
- J12 pad 1: /SENS_M -> /+12V
- J12 pad 2: /GND -> /SIG2
- J12 pad 3: /SIG2 -> /GND
- J12 pad 4: /+12V -> /SENS_M
- J13 pad 1: /SENS_M -> /+12V
- J13 pad 2: /GND -> /SIG3
- J13 pad 3: /SIG3 -> /GND
- J13 pad 4: /+12V -> /SENS_M
- J14 pad 1: /SENS_M -> /+12V
- J14 pad 2: /GND -> /SIG4
- J14 pad 3: /SIG4 -> /GND
- J14 pad 4: /+12V -> /SENS_M
- J15 pad 1: /SENS_M -> /+12V
- J15 pad 2: /GND -> /SIG5
- J15 pad 3: /SIG5 -> /GND
- J15 pad 4: /+12V -> /SENS_M
- J16 pad 1: /SENS_M -> /+12V
- J16 pad 2: /GND -> /SIG6
- J16 pad 3: /SIG6 -> /GND
- J16 pad 4: /+12V -> /SENS_M
- J17 pad 1: /SENS_M -> /+12V
- J17 pad 2: /GND -> /SIG7
- J17 pad 3: /SIG7 -> /GND
- J17 pad 4: /+12V -> /SENS_M
- J18 pad 1: /SENS_M -> /+12V
- J18 pad 2: /GND -> /SIG8
- J18 pad 3: /SIG8 -> /GND
- J18 pad 4: /+12V -> /SENS_M
- J4 pad 1: /GND -> /+3V3
- J4 pad 2: /+3V3 -> /GND
- J4 pad 3: /MCP_INTA -> /MCP_INTB
- J4 pad 4: /MCP_INTB -> /MCP_INTA
- J7 pad 1: /MCP_INTA -> /MCP_INTB
- J7 pad 2: /MCP_INTB -> /MCP_INTA
Routing:
- net /SDA_J1: track 0.00 -> 31.9 mm
- net /+12V_FILT: track 16.7 -> 47.2 mm
- net /GND: track 307.3 -> 333.4 mm
- net /+12V_RAW: track 16.7 -> 42.5 mm
- net /SCL_J1: track 0.00 -> 24.2 mm
- net /SCL: track 116.3 -> 94.2 mm
- net /SDA: track 126.2 -> 105.4 mm, vias 2 -> 0
- net /+12V: track 152.9 -> 169.8 mm
- net /LED_A: track 0.00 -> 8.80 mm
- net /MCP_INTB: track 37.8 -> 33.4 mm
- net /MCP_INTA: track 33.4 -> 37.8 mm
- net /+3V3: track 185.7 -> 187.8 mm
- net /MCP_RST: track 8.13 -> 9.78 mm
- net /+12V_SEL: track 14.2 -> 13.3 mm
Other:
- board text added: "3.3"
- board text added: "3.3V"
- board text added: "A0"
- board text added: "A1"
- board text added: "A2"
- board text added: "A3"
- board text added: "A4"
- board text added: "A5"
- board text added: "A6"
- board text added: "A7"
- board text added: "B0"
- board text added: "B1"
- board text added: "B2"
- board text added: "B3"
- board text added: "B4"
- board text added: "B5"
- board text added: "B6"
- board text added: "B7"
- board text added: "FreeZanz Evolution Connect I/O 20260915v02"
- board text added: "GND"
- board text added: "M Close=reverse I/O of sensors"
- board text added: "NC"
- board text added: "RST"
- board text added: "SCL"
- board text added: "SDA"
- board text removed: "FreeZanz Evolution Connect I/O 20260803v01"
