File: freezanz-level-io/freezanz-level-io.kicad_sch (KiCad schematic)
At the start: 51 parts, among them J1 IDC 2x4 <- Freezanz J3, J11 S1, J12 S2, J13 S3, J14 S4, J15 S5, J16 S6, J17 S7, J18 S8, J21 I2C EXP1, J22 I2C EXP2, J23 I2C EXP3, J3 MCP LEFT, J4 MCP RIGHT, J6 PORT B, J7 INT / SPARE, J8 GPIO5 OUT, J9 GPIO15 OUT

Commit message: Pushing v2 version of the breakout board
Parts:
- added D2: LED, LED_THT:LED_D5.0mm, symbol Device:LED
- added R6, R7: 470R, Resistor_THT:R_Axial_DIN0207_L6.3mm_D2.5mm_P7.62mm_Horizontal, symbol Device:R
- added R8: 10k, Resistor_THT:R_Axial_DIN0207_L6.3mm_D2.5mm_P7.62mm_Horizontal, symbol Device:R
Connections:
- net +12V: now also J11.1 (Pin_1), J12.1 (Pin_1), J13.1 (Pin_1), J14.1 (Pin_1), J15.1 (Pin_1), J16.1 (Pin_1), J17.1 (Pin_1), J18.1 (Pin_1), R8.1; no longer J11.4 (Pin_4), J12.4 (Pin_4), J13.4 (Pin_4), J14.4 (Pin_4), J15.4 (Pin_4), J16.4 (Pin_4), J17.4 (Pin_4), J18.4 (Pin_4)
- net +3V3: now also J4.1 (Pin_1); no longer J4.2 (Pin_2)
- net GND: now also J11.3 (Pin_3), J12.3 (Pin_3), J13.3 (Pin_3), J14.3 (Pin_3), J15.3 (Pin_3), J16.3 (Pin_3), J17.3 (Pin_3), J18.3 (Pin_3), J4.2 (Pin_2), D2.1 (K); no longer J11.2 (Pin_2), J12.2 (Pin_2), J13.2 (Pin_2), J14.2 (Pin_2), J15.2 (Pin_2), J16.2 (Pin_2), J17.2 (Pin_2), J18.2 (Pin_2), J4.1 (Pin_1)
- net MCP_INTA: now also J4.4 (Pin_4), J7.2 (Pin_2); no longer J4.3 (Pin_3), J7.1 (Pin_1)
- net MCP_INTB: now also J4.3 (Pin_3), J7.1 (Pin_1); no longer J4.4 (Pin_4), J7.2 (Pin_2)
- net SCL: now also R7.2; no longer J1.7 (Pin_7)
- net SDA: now also R6.2; no longer J1.5 (Pin_5)
- net SENS_M: now also J11.4 (Pin_4), J12.4 (Pin_4), J13.4 (Pin_4), J14.4 (Pin_4), J15.4 (Pin_4), J16.4 (Pin_4), J17.4 (Pin_4), J18.4 (Pin_4); no longer J11.1 (Pin_1), J12.1 (Pin_1), J13.1 (Pin_1), J14.1 (Pin_1), J15.1 (Pin_1), J16.1 (Pin_1), J17.1 (Pin_1), J18.1 (Pin_1)
- net SIG1: now also J11.2 (Pin_2); no longer J11.3 (Pin_3)
- net SIG2: now also J12.2 (Pin_2); no longer J12.3 (Pin_3)
- net SIG3: now also J13.2 (Pin_2); no longer J13.3 (Pin_3)
- net SIG4: now also J14.2 (Pin_2); no longer J14.3 (Pin_3)
- net SIG5: now also J15.2 (Pin_2); no longer J15.3 (Pin_3)
- net SIG6: now also J16.2 (Pin_2); no longer J16.3 (Pin_3)
- net SIG7: now also J17.2 (Pin_2); no longer J17.3 (Pin_3)
- net SIG8: now also J18.2 (Pin_2); no longer J18.3 (Pin_3)
- net GPB0 renamed A0
- net GPB1 renamed A1
- net GPB2 renamed A2
- net GPB3 renamed A3
- net GPB4 renamed A4
- net GPB5 renamed A5
- net GPB6 renamed A6
- net GPB7 renamed A7
- net IO1 renamed B0
- net IO2 renamed B1
- net IO3 renamed B2
- net IO4 renamed B3
- net IO5 renamed B4
- net IO6 renamed B5
- net IO7 renamed B6
- net IO8 renamed B7
- new net LED_A: D2.2 (A), R8.2
- new net SCL_J1: J1.7 (Pin_7), R7.1
- new net SDA_J1: J1.5 (Pin_5), R6.1
